Commit message: 修正IMU的重力

File: legged_examples/lion_description/robot.xacro (robot description, xacro)
@@ -8,4 +8,5 @@
     <!-- <xacro:include filename="$(find lion_description)/urdf/$(arg robot_type)/const.xacro"/> -->
         <!--Robot Model*******************************************************************************************-->
+        <!-- <link name="world"/> -->
         <link name="base">
           <inertial>
@@ -30,4 +31,8 @@
           </collision>
         </link>
+        <!-- <joint name="base_to_world" type="fixed">
+          <parent link="world"/>
+          <child link="base"/>
+        </joint> -->
         <link name="RF_hip">
           <inertial>
