Commit message: 添加末端执行器topic有问题

File: legged_examples/lion_armed_description/robot.xacro (robot description, xacro)
@@ -641,6 +641,6 @@
         lower="-2.618"
         upper="2.618"
-        effort="15.0"
-        velocity="20.0" />
+        effort="25.0"
+        velocity="10.0" />
     </joint>
     <link name="upper_arm_link">
@@ -693,6 +693,6 @@
         lower="0"
         upper="3.665"
-        effort="15.0"
-        velocity="20.0" />
+        effort="25.0"
+        velocity="10.0" />
     </joint>
     <link name="elbow_link">
@@ -745,6 +745,6 @@
         lower="0"
         upper="4.188"
-        effort="15.0"
-        velocity="20.0" />
+        effort="25.0"
+        velocity="10.0" />
     </joint>
     <link name="lower_arm_link">
@@ -795,8 +795,9 @@
         xyz="-1 0 0" />
       <limit
-        lower="-3.14"
-        upper="3.14"
+        lower="-3."
+        upper="3."
         effort="15.0"
-        velocity="20.0" />
+        velocity="10.0" />
+      <dynamics damping="0.1" friction="0.01"/>
     </joint>
     <link name="wrist_link">
@@ -850,5 +851,6 @@
         upper="1.571"
         effort="15.0"
-        velocity="20.0" />
+        velocity="10.0" />
+      <dynamics damping="0.1" friction="0.01"/>
     </joint>
     <link name="hand_link">
@@ -899,8 +901,9 @@
         xyz="1 0 0" />
       <limit
-        lower="-3.14"
-        upper="3.14"
+        lower="-10."
+        upper="10."
         effort="15.0"
-        velocity="20.0" />
+        velocity="10.0" />
+      <dynamics damping="0.1" friction="0.01"/>
     </joint>
     <xacro:IMU connected_to="base" imu_name="unitree_imu" xyz="0. 0. 0." rpy="0. 0. 0."/>

Commit message: adjust with arm

File: legged_examples/lion_armed_description/robot.xacro (robot description, xacro)
@@ -638,4 +638,5 @@
       <axis
         xyz="0 0 -1" />
+      <dynamics damping="0.3"/>
       <limit
         lower="-2.618"
@@ -690,4 +691,5 @@
       <axis
         xyz="0 1 0" />
+      <dynamics damping="0.2"/>
       <limit
         lower="0"
@@ -742,4 +744,5 @@
       <axis
         xyz="0 -1 0" />
+      <dynamics damping="0.2"/>
       <limit
         lower="0"

Commit message: using inverse dynamics ,not wbc

File: legged_examples/lion_armed_description/robot.xacro (robot description, xacro)
@@ -744,5 +744,5 @@
       <axis
         xyz="0 -1 0" />
-      <dynamics damping="0.2"/>
+      <dynamics damping="0.1"/>
       <limit
         lower="0"

Commit message: using another wbc from skywoods; remove ee wrench

File: legged_examples/lion_armed_description/robot.xacro (robot description, xacro)
@@ -638,5 +638,5 @@
       <axis
         xyz="0 0 -1" />
-      <dynamics damping="0.3"/>
+      <dynamics damping="0.1" friction="0.01"/>
       <limit
         lower="-2.618"
@@ -691,5 +691,5 @@
       <axis
         xyz="0 1 0" />
-      <dynamics damping="0.2"/>
+      <dynamics damping="0.1" friction="0.01"/>
       <limit
         lower="0"
@@ -744,5 +744,5 @@
       <axis
         xyz="0 -1 0" />
-      <dynamics damping="0.1"/>
+      <dynamics damping="0.1" friction="0.01"/>
       <limit
         lower="0"
@@ -851,6 +851,6 @@
         xyz="0 -1 0" />
       <limit
-        lower="-1.571"
-        upper="1.571"
+        lower="-1."
+        upper="1."
         effort="15.0"
         velocity="10.0" />

Commit message: remove hierarchical wbc

File: legged_examples/lion_armed_description/robot.xacro (robot description, xacro)
@@ -802,5 +802,5 @@
         effort="15.0"
         velocity="10.0" />
-      <dynamics damping="0.1" friction="0.01"/>
+      <dynamics damping="0.1" friction="0.2"/>
     </joint>
     <link name="wrist_link">
@@ -855,5 +855,5 @@
         effort="15.0"
         velocity="10.0" />
-      <dynamics damping="0.1" friction="0.01"/>
+      <dynamics damping="0.1" friction="0.2"/>
     </joint>
     <link name="hand_link">
@@ -908,5 +908,5 @@
         effort="15.0"
         velocity="10.0" />
-      <dynamics damping="0.1" friction="0.01"/>
+      <dynamics damping="0.1" friction="0.2"/>
     </joint>
     <xacro:IMU connected_to="base" imu_name="unitree_imu" xyz="0. 0. 0." rpy="0. 0. 0."/>
