Commit message: simplify arx arm collision model

File: legged_examples/lion_arx_description/robot.xacro (robot description, xacro)
@@ -589,10 +589,8 @@
     </visual>
     <collision>
-      <origin
-        xyz="0 0 0"
-        rpy="0 0 0" />
-      <geometry>
-        <mesh
-          filename="package://lion_arx_description/meshes/arm_base_link.STL" />
+      <origin rpy="0 0 0" xyz="0 0.0 0.03" />
+      <geometry>
+        <!-- <box size="0.05 0.03 0.3"/> -->
+        <cylinder length="0.05" radius="0.03" />
       </geometry>
     </collision>
@@ -641,6 +639,5 @@
         rpy="0 0 0" />
       <geometry>
-        <mesh
-          filename="package://lion_arx_description/meshes/link1.STL" />
+        <cylinder length="0.01" radius="0.03" />
       </geometry>
     </collision>
@@ -694,10 +691,8 @@
     </visual>
     <collision>
-      <origin
-        xyz="0 0 0"
-        rpy="0 0 0" />
-      <geometry>
-        <mesh
-          filename="package://lion_arx_description/meshes/link2.STL" />
+      <origin rpy="0 ${pi/2.0} 0" xyz="-0.14 0.0 0.0" />
+      <geometry>
+        <!-- <box size="0.05 0.03 0.3"/> -->
+        <cylinder length="0.28" radius="0.025" />
       </geometry>
     </collision>
@@ -751,10 +746,8 @@
     </visual>
     <collision>
-      <origin
-        xyz="0 0 0"
-        rpy="0 0 0" />
-      <geometry>
-        <mesh
-          filename="package://lion_arx_description/meshes/link3.STL" />
+      <origin rpy="0 ${pi/2.0} 0" xyz="0.15 0.0 -0.055" />
+      <geometry>
+        <!-- <box size="0.05 0.03 0.3"/> -->
+        <cylinder length="0.2" radius="0.02" />
       </geometry>
     </collision>
@@ -808,10 +801,8 @@
     </visual>
     <collision>
-      <origin
-        xyz="0 0 0"
-        rpy="0 0 0" />
-      <geometry>
-        <mesh
-          filename="package://lion_arx_description/meshes/link4.STL" />
+      <origin rpy="${pi/2.0} 0 0" xyz="0.06 0.0 -0.0" />
+      <geometry>
+        <!-- <box size="0.05 0.03 0.3"/> -->
+        <cylinder length="0.06" radius="0.025" />
       </geometry>
     </collision>
@@ -865,10 +856,8 @@
     </visual>
     <collision>
-      <origin
-        xyz="0 0 0"
-        rpy="0 0 0" />
-      <geometry>
-        <mesh
-          filename="package://lion_arx_description/meshes/link5.STL" />
+      <origin rpy="0 ${pi/2.0} 0" xyz="0.06 0.0 -0.0" />
+      <geometry>
+        <!-- <box size="0.05 0.03 0.3"/> -->
+        <cylinder length="0.06" radius="0.025" />
       </geometry>
     </collision>
