Commit message: add base frame rotation to end effector pos control

File: legged_examples/lion_arx_description/lion_arx.urdf (robot description, URDF)
Before this commit: robot lion, 25 links, 24 joints
Joints:
- joint joint3: limit lower=0. upper=3.14 effort=25. velocity=10. -> lower=0.05 upper=3.14 effort=25. velocity=10.

File: legged_examples/lion_arx_description/robot.xacro (robot description, xacro)
@@ -765,5 +765,5 @@
       xyz="0 1 0" />
     <limit
-      lower="0."
+      lower="0.05"
       upper="3.14"
       effort="25."

Commit message: modify end effector's model to a gripper

File: legged_examples/lion_arx_description/lion_arx.urdf (robot description, URDF)
Before this commit: robot lion, 25 links, 24 joints
Links:
- link arm_base_link: geometry collision cylinder length=0.05 radius=0.03; visual mesh filename=package://lion_arx_description/meshes/arm_base_link.STL
- link elbow_link: geometry collision cylinder length=0.2 radius=0.02; visual mesh filename=package://lion_arx_description/meshes/link3.STL
- link hand_link: geometry collision cylinder length=0.1 radius=0.01; visual mesh filename=package://lion_arx_description/meshes/link6.STL
- link lower_arm_link: geometry collision cylinder length=0.06 radius=0.025; visual mesh filename=package://lion_arx_description/meshes/link4.STL
- link shoulder_link: geometry collision cylinder length=0.01 radius=0.03; visual mesh filename=package://lion_arx_description/meshes/link1.STL
- link upper_arm_link: geometry collision cylinder length=0.28 radius=0.025; visual mesh filename=package://lion_arx_description/meshes/link2.STL
- link wrist_link: geometry collision cylinder length=0.06 radius=0.025; visual mesh filename=package://lion_arx_description/meshes/link5.STL

File: legged_examples/lion_arx_description/robot.xacro (robot description, xacro)
@@ -912,9 +912,8 @@
     <collision>
       <origin
-        xyz="0 0 0"
-        rpy="0 0 0" />
-      <geometry>
-        <mesh
-          filename="package://lion_arx_description/meshes/link6.STL" />
+        xyz="0.07 0 0"
+        rpy="0 ${pi/2.0} 0" />
+      <geometry>
+        <cylinder length="0.14" radius="0.01" />
       </geometry>
     </collision>
