Commit message: add: 3 dof arm control realized in simulation

File: legged_examples/lion_arx3_description/robot.xacro (robot description, xacro)
@@ -659,5 +659,5 @@
       effort="25.0"
       velocity="10.0" />
-    <dynamics damping="0.1" friction="0.01"/>
+    <dynamics damping="0.3" friction="0.1"/>
   </joint>
   <link name="upper_arm_link">

Commit message: add: arm ee pos constrol in mpc

File: legged_examples/lion_arx3_description/robot.xacro (robot description, xacro)
@@ -769,5 +769,5 @@
       effort="25."
       velocity="10." />
-    <dynamics damping="0.1" friction="0.01"/>
+    <dynamics damping="0.3" friction="0.01"/>
   </joint>
   <link name="lower_arm_link">
